File: kicad/v0.1/NextTRS.kicad_sch (KiCad schematic)
At the start: 97 parts, among them J1 TRS-80 M3 Pin Header, J10 AudioJack3, J11 Mini-DIN-6, J12 USB_B_Micro, J2 TRS-80 M1 Pin Connector, J3 TRS-80 M3 Edge Connector, J4 TRS-80 M1 Edge Connector, J5 Conn_01x06_Male, J6 Conn_01x06_Male, J7 HDMI_A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

Commit message: New routing for U5
Connections:
- net CTRL1_EN: now also Conn1.182 (D10); no longer Conn1.192 (R7)
- net EXTIOSEL_IN_N: now also Conn1.186 (E10); no longer Conn1.194 (P7)
- net GND: now also U5.8 (A6), U5.9 (A7)
- net HSYNC: now also U5.7 (A5); no longer U5.5 (A3)
- net HSYNCX: now also Conn1.200 (L8), U5.13 (B5); no longer Conn1.182 (D10), U5.15 (B3)
- net INT_IN_N: now also Conn1.194 (P7); no longer Conn1.200 (L8)
- net VIDEO: now also U5.5 (A3); no longer U5.7 (A5)
- net VIDEOX: now also U5.15 (B3); no longer U5.13 (B5)
- net VSYNCX: now also Conn1.198 (M6); no longer Conn1.186 (E10)
- net WAIT_IN_N: now also Conn1.192 (R7); no longer Conn1.198 (M6)
